File: pcbs/corne-indian/corne-inidan-hotswap/left.kicad_sch (KiCad schematic)
At the start: 10 parts, among them SW1 SW_Push

Commit message: Left side LED & switch schematic added But need to check
Parts:
- added LED1, LED10, LED11, LED12, LED13, LED14, LED15, LED16, LED17, LED18, LED19, LED2, LED20, LED21, LED3, LED4, LED5, LED6, LED7, LED8, LED9: SK6812MINI-E, User_Button_Switch_Keyboard:YS-SK6812MINI-E, symbol LED_RGB:LED_SK6812MINI-E
- added SW10, SW11, SW12, SW13, SW14, SW15, SW16, SW17, SW18, SW19, SW2, SW20, SW21, SW3, SW4, SW5, SW6, SW7, SW8, SW9: SW_Push, User_Button_Switch_Keyboard:SW_Cherry_MX_1.00u_Hotswap, symbol Switch:SW_Push
- SW1: footprint Button_Switch_Keyboard:SW_Cherry_MX_1.50u_PCB -> User_Button_Switch_Keyboard:SW_Cherry_MX_1.50u_Hotswap
- renumbered GSM1 to MCU1
Connections:
- net GND: now also SW1.2, LED1.3 (VSS), LED10.3 (VSS), LED11.3 (VSS), LED12.3 (VSS), LED13.3 (VSS), LED14.3 (VSS), LED15.3 (VSS), LED16.3 (VSS), LED17.3 (VSS), LED18.3 (VSS), LED19.3 (VSS), LED2.3 (VSS), LED20.3 (VSS), LED21.3 (VSS), LED3.3 (VSS), LED4.3 (VSS), LED5.3 (VSS), LED6.3 (VSS), LED7.3 (VSS), LED8.3 (VSS), LED9.3 (VSS), SW10.2, SW11.2, SW12.2, SW13.2, SW14.2, SW15.2, SW16.2, SW17.2, SW18.2, SW19.2, SW2.2, SW20.2, SW21.2, SW3.2, SW4.2, SW5.2, SW6.2, SW7.2, SW8.2, SW9.2
- net KEY_1: now reaches SW1.1
- new net 5V_L: LED1.1 (VDD), LED10.1 (VDD), LED11.1 (VDD), LED12.1 (VDD), LED13.1 (VDD), LED14.1 (VDD), LED15.1 (VDD), LED16.1 (VDD), LED17.1 (VDD), LED18.1 (VDD), LED19.1 (VDD), LED2.1 (VDD), LED20.1 (VDD), LED21.1 (VDD), LED3.1 (VDD), LED4.1 (VDD), LED5.1 (VDD), LED6.1 (VDD), LED7.1 (VDD), LED8.1 (VDD), LED9.1 (VDD)
- new net KEY_10: SW10.1
- new net KEY_11: SW11.1
- new net KEY_12: SW12.1
- new net KEY_13: SW13.1
- new net KEY_14: SW14.1
- new net KEY_15: SW15.1
- new net KEY_16: SW16.1
- new net KEY_17: SW17.1
- new net KEY_18: SW18.1
- new net KEY_19: SW19.1
- new net KEY_2: SW2.1
- new net KEY_20: SW20.1
- new net KEY_21: SW21.1
- new net KEY_3: SW3.1
- new net KEY_4: SW4.1
- new net KEY_5: SW5.1
- new net KEY_6: SW6.1
- new net KEY_7: SW7.1
- new net KEY_8: SW8.1
- new net KEY_9: SW9.1
- new net L_KEY: LED1.4 (DIN)
- new net L_KEY10: LED10.4 (DIN), LED9.2 (DOUT)
- new net L_KEY11: LED10.2 (DOUT), LED11.4 (DIN)
- new net L_KEY12: LED11.2 (DOUT), LED12.4 (DIN)
- new net L_KEY13: LED12.2 (DOUT), LED13.4 (DIN)
- new net L_KEY14: LED13.2 (DOUT), LED14.4 (DIN)
- new net L_KEY15: LED14.2 (DOUT), LED15.4 (DIN)
- new net L_KEY16: LED15.2 (DOUT), LED16.4 (DIN)
- new net L_KEY17: LED16.2 (DOUT), LED17.4 (DIN)
- new net L_KEY18: LED17.2 (DOUT), LED18.4 (DIN)
- new net L_KEY19: LED18.2 (DOUT), LED19.4 (DIN)
- new net L_KEY2: LED1.2 (DOUT), LED2.4 (DIN)
- new net L_KEY20: LED19.2 (DOUT), LED20.4 (DIN)
- new net L_KEY21: LED20.2 (DOUT), LED21.4 (DIN)
- new net L_KEY22: LED21.2 (DOUT)
- new net L_KEY3: LED2.2 (DOUT), LED3.4 (DIN)
- new net L_KEY4: LED3.2 (DOUT), LED4.4 (DIN)
- new net L_KEY5: LED4.2 (DOUT), LED5.4 (DIN)
- new net L_KEY6: LED5.2 (DOUT), LED6.4 (DIN)
- new net L_KEY7: LED6.2 (DOUT), LED7.4 (DIN)
- new net L_KEY8: LED7.2 (DOUT), LED8.4 (DIN)
- new net L_KEY9: LED8.2 (DOUT), LED9.4 (DIN)
Other:
- moved on the sheet: D1, MCU1, R1, R2, R3, R5, SW1, TP10, TP3, TP9
