File: pcbs/corne-indian/corne-inidan-hotswap/corne-inidan-hotswap.kicad_pcb (KiCad board)
At the start: 2 copper layers, 277.2 x 107.5 mm, 209 parts, among them J1 Conn_01x03_Pin, J2 Conn_01x04_Pin, J3 PJ-3136-B, J4 USB_A, J5 USB4105 - Type C USB 2.0 Conn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, J6 USB_A, J7 USB_A, J8 USB_A, Q1 SI2301, SW1 SW_Push, SW10 SW_Push, SW11 SW_Push, SW12 SW_Push, SW13 SW_Push, SW14 SW_Push, SW15 SW_Push, SW16 SW_Push, SW17 SW_Push, SW18 SW_Push, SW19 SW_Push, SW2 SW_Push, SW20 SW_Push, SW21 SW_Push, SW3 SW_Push, SW4 SW_Push, SW5 SW_Push, SW6 SW_Push, SW7 SW_Push, SW8 SW_Push, SW9 SW_Push, U1 AP2127K-3.3, U2 RP2040, U3 W25Q32JVSS, U4 AMS1117-3.3, U5 CH334F, Y1 12Mhz, Y2 12Mhz

Commit message: Mid of the Layout
Parts:
- C7, R7, R9, TP2, TP3: moved to B.Cu
- moved C10 131.1 mm to (111.8, 210.8)
- moved C11 131.1 mm to (111.8, 213.3)
- moved C9 131.1 mm to (111.8, 208.2)
- moved R8 131.1 mm to (118.3, 210.2)
- moved R9 89.8 mm to (135.0, 172.5), turned to -90 degrees
- moved R7 84.3 mm to (104.8, 156.2)
- moved TP2 53.5 mm to (179.8, 129.2), turned to 180 degrees
- moved TP3 44.1 mm to (179.0, 121.5), turned to 180 degrees
- moved C7 7.07 mm to (105.8, 154.0), turned to -90 degrees
Connections:
- J2 pad 3: /left/SCL -> /left/REB
- J2 pad 4: /left/SDA -> /left/RE1A
- rJ2 pad 3: /Right/SCL -> /Right/REB
- rJ2 pad 4: /Right/SDA -> /Right/RE1A
Routing:
- net /left/U_-: track 0.00 -> 126.8 mm
- net /left/U_+: track 0.00 -> 125.9 mm
- net /left/KEY_21: track 1.62 -> 59.3 mm
- net /left/KEY_EX2: track 0.00 -> 47.1 mm
- net /left/KEY_20: track 1.58 -> 39.9 mm
- net /left/KEY_16: track 2.45 -> 38.6 mm, vias 0 -> 2
- net /left/KEY_17: track 1.62 -> 37.2 mm, vias 0 -> 1
- net Net-(U2-GPIO21): track 1.62 -> 22.8 mm
- net /left/KEY_18: track 1.58 -> 22.8 mm
- net /left/KEY_EX1: track 0.00 -> 18.5 mm
- net /left/RE0A: track 0.00 -> 18.4 mm
- net /left/RE1A: track 0.00 -> 18.4 mm
- net /left/REB: track 0.00 -> 18.3 mm
- net /left/USB_VBUS_PIN: track 0.00 -> 17.7 mm
- net /left/KEY_3: track 1.73 -> 18.8 mm
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
Commit message: Mid of the routing
Parts:
- C10, C11, R8, rC10, rC11, rC7, rC9, rR7: moved to B.Cu
- moved rR8 106.7 mm to (274.5, 170.7)
- moved rR9 106.7 mm to (274.5, 173.2)
- moved rC9 103.1 mm to (272.8, 156.8), turned to 90 degrees
- moved rC10 91.0 mm to (241.8, 163.2)
- moved rR7 90.3 mm to (247.8, 163.2), turned to 180 degrees
- moved rC11 89.8 mm to (244.8, 163.2), turned to 180 degrees
- moved rC7 83.6 mm to (253.8, 156.2)
- moved C9 57.7 mm to (127.5, 152.8)
- moved C10 57.3 mm to (104.2, 154.0), turned to -90 degrees
- moved C11 56.9 mm to (107.8, 156.5), turned to 180 degrees
- moved rTP1 45.9 mm to (197.4, 89.2), turned to 90 degrees
- moved R8 44.2 mm to (137.2, 170.2), turned to 180 degrees
- moved TP5 41.0 mm to (201.4, 89.2), turned to 90 degrees
- moved TP6 37.4 mm to (204.5, 89.2), turned to 90 degrees
Routing:
- net /left/KEY_19: track 0.00 -> 105.3 mm, vias 0 -> 8
- net /Right/U_+: track 0.00 -> 91.2 mm, vias 0 -> 2
- net /Right/U_-: track 0.00 -> 90.1 mm, vias 0 -> 2
- net /left/KEY_13: track 0.00 -> 58.6 mm, vias 0 -> 4
- net /Right/KEY_EX2: track 0.00 -> 54.1 mm
- net /Right/RE0A: track 0.00 -> 53.9 mm
- net /Right/KEY_EX1: track 0.00 -> 53.5 mm
- net /left/KEY_14: track 0.00 -> 50.7 mm, vias 0 -> 2
- net /Right/KEY_2: track 0.00 -> 48.7 mm
- net /left/KEY_20: track 39.9 -> 88.4 mm, vias 0 -> 4
- net /Right/KEY_21: track 0.00 -> 43.2 mm, vias 0 -> 1
- net /left/RE1A: track 18.4 -> 50.4 mm
- net /left/RE0A: track 18.4 -> 50.5 mm
- net /left/KEY_15: track 0.00 -> 31.5 mm
- net +3.3V: track 94.7 -> 126.1 mm, vias 5 -> 7
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
Commit message: Still layouting & mid of the Routing is going on
Parts:
- moved rR8 0.24 mm to (274.5, 170.5)
Routing:
- net /Right/KEY_5: track 12.4 -> 85.9 mm
- net /Right/KEY_12: track 13.1 -> 69.8 mm
- net /Right/KEY_11: track 11.7 -> 59.7 mm
- net /Right/RE1A: track 0.00 -> 43.9 mm, vias 0 -> 2
- net /Right/KEY_13: track 13.8 -> 53.0 mm, vias 0 -> 2
- net /Right/REB: track 0.00 -> 34.6 mm, vias 0 -> 2
- net /Right/KEY_3: track 34.3 -> 67.3 mm, vias 0 -> 2
- net /Right/KEY_4: track 34.4 -> 64.9 mm, vias 0 -> 2
- net /Right/KEY_6: track 30.5 -> 53.3 mm, vias 0 -> 2
- net /Right/KEY_14: track 14.6 -> 33.6 mm
- net GND: track 40.3 -> 56.3 mm, vias 26 -> 29
- net /Right/KEY_16: track 1.69 -> 17.4 mm
- net /Right/KEY_15: track 0.00 -> 14.8 mm
- net +5V: track 0.00 -> 14.1 mm, vias 0 -> 1
- net /Right/RESET: track 7.24 -> 19.4 mm
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