File: pcbs/corne-indian/corne-inidan-hotswap/corne-inidan-hotswap.kicad_pcb (KiCad board)
At the start: 2 copper layers, 277.2 x 107.5 mm, 209 parts, among them J1 Conn_01x03_Pin, J2 Conn_01x04_Pin, J3 PJ-3136-B, J4 USB_A, J5 USB4105 - Type C USB 2.0 Conn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, J6 USB_A, J7 USB_A, J8 USB_A, Q1 SI2301, SW1 SW_Push, SW10 SW_Push, SW11 SW_Push, SW12 SW_Push, SW13 SW_Push, SW14 SW_Push, SW15 SW_Push, SW16 SW_Push, SW17 SW_Push, SW18 SW_Push, SW19 SW_Push, SW2 SW_Push, SW20 SW_Push, SW21 SW_Push, SW3 SW_Push, SW4 SW_Push, SW5 SW_Push, SW6 SW_Push, SW7 SW_Push, SW8 SW_Push, SW9 SW_Push, U1 AP2127K-3.3, U2 RP2040, U3 W25Q32JVSS, U4 AMS1117-3.3, U5 CH334F, Y1 12Mhz, Y2 12Mhz

Commit message: Mid of the Routing almost done for Switch & then Still LED not started
Parts:
- added ?: , , F.Cu at (277.0, 101.2)
- added ?: , , F.Cu at (278.0, 101.2)
- added ?: , , F.Cu at (98.0, 101.2)
- added ?: , , F.Cu at (79.0, 165.2)
- added ?: , , F.Cu at (279.0, 101.2)
- added ?: , , F.Cu at (81.0, 165.2)
- added ?: , , F.Cu at (80.0, 165.2)
- added ?: , , F.Cu at (316.2, 165.2)
- added ?: , , F.Cu at (96.0, 101.2)
- added ?: , , F.Cu at (59.0, 165.2)
- added ?: , , F.Cu at (315.2, 165.2)
- added ?: , , F.Cu at (296.0, 165.2)
- added ?: , , F.Cu at (300.0, 165.2)
- added ?: , , F.Cu at (281.0, 101.2)
- added ?: , , F.Cu at (319.2, 165.2)
- added ?: , , F.Cu at (297.0, 165.2)
- added ?: , , F.Cu at (99.0, 101.2)
- added ?: , , F.Cu at (61.0, 165.2)
- added ?: , , F.Cu at (239.0, 101.2)
- added ?: , , F.Cu at (134.2, 101.2)
- added ?: , , F.Cu at (135.2, 101.2)
- added ?: , , F.Cu at (58.0, 165.2)
- added ?: , , F.Cu at (240.0, 101.2)
- added ?: , , F.Cu at (280.0, 101.2)
- added ?: , , F.Cu at (241.0, 101.2)
- added ?: , , F.Cu at (97.0, 101.2)
- added ?: , , F.Cu at (136.2, 101.2)
- added ?: , , F.Cu at (60.0, 165.2)
- added ?: , , F.Cu at (318.2, 165.2)
- added ?: , , F.Cu at (242.0, 101.2)
- added ?: , , F.Cu at (78.0, 165.2)
- added ?: , , F.Cu at (62.0, 165.2)
- added ?: , , F.Cu at (77.0, 165.2)
- added ?: , , F.Cu at (298.0, 165.2)
- added ?: , , F.Cu at (317.2, 165.2)
- added ?: , , F.Cu at (243.0, 101.2)
- added ?: , , F.Cu at (138.2, 101.2)
- added ?: , , F.Cu at (100.0, 101.2)
- added ?: , , F.Cu at (299.0, 165.2)
- added ?: , , F.Cu at (137.2, 101.2)
- added D6: DSK34, Diode_SMD:D_SOD-123F, F.Cu at (167.5, 88.5)
- added rD6: DSK34, Diode_SMD:D_SOD-123F, F.Cu at (217.5, 90.0)
- C9, rR8, rR9: moved to B.Cu
- moved C19 321.4 mm to (363.3, 114.8), turned to 0 degrees
- moved C21 317.6 mm to (363.3, 117.8), turned to 0 degrees
- moved J5 314.1 mm to (367.0, 152.7), turned to 0 degrees
- moved C18 314.1 mm to (363.1, 138.6), turned to 0 degrees
- moved C24 313.8 mm to (363.3, 120.8), turned to 0 degrees
- moved R13 312.6 mm to (371.1, 141.1)
- moved C20 311.1 mm to (363.1, 141.1), turned to 0 degrees
- moved C25 310.1 mm to (363.3, 123.8), turned to 0 degrees
- moved D2 309.9 mm to (368.3, 114.9), turned to 0 degrees
- moved R12 309.5 mm to (371.1, 138.6)
- moved C30 308.2 mm to (367.1, 138.6), turned to 0 degrees
- moved C22 308.1 mm to (363.1, 143.6), turned to 0 degrees
- moved C26 306.4 mm to (363.3, 126.8), turned to 0 degrees
- moved R11 306.3 mm to (367.1, 146.1)
- moved R10 306.1 mm to (367.1, 143.6)
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Routing:
- net /Right/5V_L: track 0.00 -> 95.1 mm, vias 0 -> 4
- net /Right/KEY_19: track 4.19 -> 94.5 mm, vias 0 -> 2
- net /Right/REB: track 34.6 -> 117.9 mm, vias 2 -> 6
- net +3.3V: track 136.2 -> 210.3 mm, vias 7 -> 13
- net /left/KEY_EX1: track 18.5 -> 91.5 mm, vias 0 -> 2
- net /Right/L_KEY: track 8.95 -> 78.9 mm, vias 1 -> 2
- net /left/KEY_4: track 7.10 -> 76.9 mm, vias 0 -> 4
- net /Right/KEY_EX1: track 53.5 -> 123.1 mm, vias 0 -> 2
- net /Right/KEY_18: track 4.64 -> 72.3 mm, vias 0 -> 2
- net /left/KEY_5: track 3.00 -> 66.4 mm, vias 0 -> 4
- net /left/KEY_12: track 4.12 -> 67.5 mm, vias 0 -> 2
- net /left/REB: track 47.1 -> 103.5 mm, vias 0 -> 1
- net /Right/KEY_20: track 20.5 -> 75.4 mm, vias 0 -> 4
- net VBUS: track 23.7 -> 76.4 mm, vias 2 -> 5
- net +5V: track 14.1 -> 65.4 mm, vias 1 -> 3
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