File: pcbs/corne-indian/corne-inidan-hotswap/Right.kicad_sch (KiCad schematic)
At the start: 88 parts

Commit message: left side Layout of the Keyboard is done
Partial side of the right design is also Done
Connections:
- net +3.3V renamed r+3.3V
- net +5V renamed r+5V
- net VBUS renamed rVBUS
Changed lines of the file:
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@@
 			)
 		)
-		(property "Value" "+3.3V"
+		(property "Value" "r+3.3V"
 			(at 163.83 26.67 0)
 			(effects
@@
 			)
 		)
-		(property "Value" "+3.3V"
+		(property "Value" "r+3.3V"
 			(at 349.25 29.21 0)
 			(effects
@@
 			)
 		)
-		(property "Value" "+3.3V"
+		(property "Value" "r+3.3V"
 			(at 157.48 52.07 0)
 			(effects
@@
 			)
 		)
-		(property "Value" "+5V"
+		(property "Value" "r+5V"
 			(at 259.08 60.96 90)
 			(effects
@@
 			)
 		)
-		(property "Value" "+5V"
+		(property "Value" "r+5V"
 			(at 123.952 52.07 0)
 			(effects
@@
 			)
 		)
-		(property "Value" "+5V"
+		(property "Value" "r+5V"
 			(at 74.93 74.168 0)
 			(effects
@@
 			)
 		)
-		(property "Value" "VBUS"
+		(property "Value" "rVBUS"
 			(at 63.5 30.48 0)
 			(effects
@@
 			)
 		)
-		(property "Value" "+5V"
+		(property "Value" "r+5V"
 			(at 89.662 31.75 0)
 			(effects
@@
 			)
 		)
-		(property "Value" "+5V"
+		(property "Value" "r+5V"
 			(at 117.602 26.67 0)
 			(effects
@@
 			)
 		)
-		(property "Value" "+3.3V"
+		(property "Value" "r+3.3V"
 			(at 342.9 158.75 0)
 			(effects
@@
 			)
 		)
-		(property "Value" "+5V"
+		(property "Value" "r+5V"
 			(at 217.17 57.15 90)
 			(effects

Commit message: PCB Layout is almost done Cosmetic Chnages need to do
Parts:
- rEXSW1, rEXSW2: footprint User_Button_Switch_Keyboard:keyswitch_cherrymx_hotswap_1u_rotary_encoder_ec12 -> User_Button_Switch_Keyboard:SW_Cherry_MX_1.00u_Hotswap_Rotary-Encoder
Changed lines of the file:
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@@
 			)
 		)
-		(property "Footprint" "User_Button_Switch_Keyboard:keyswitch_cherrymx_hotswap_1u_rotary_encoder_ec12"
+		(property "Footprint" "User_Button_Switch_Keyboard:SW_Cherry_MX_1.00u_Hotswap_Rotary-Encoder"
 			(at 53.086 154.94 0)
 			(effects
@@
 			)
 		)
-		(property "Footprint" "User_Button_Switch_Keyboard:keyswitch_cherrymx_hotswap_1u_rotary_encoder_ec12"
+		(property "Footprint" "User_Button_Switch_Keyboard:SW_Cherry_MX_1.00u_Hotswap_Rotary-Encoder"
 			(at 53.086 205.74 0)
 			(effects

Commit message: USB Circuit deleted & Design is also compeleted in LAyout level
Parts:
- added rR19: 0R, Resistor_SMD:R_0603_1608Metric, symbol Device:R
- rJ1, rU4: now not fitted; now left out of the parts list
Connections:
- net KEY_18: now also rR19.2
- net L_KEY22: now also rR19.1
Changed lines of the file:
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@@
 	(wire
 		(pts
+			(xy 99.06 96.52) (xy 106.68 96.52)
+		)
+		(stroke
+			(width 0)
+			(type default)
+		)
+	)
+	(wire
+		(pts
 			(xy 317.5 110.49) (xy 312.42 110.49)
 		)
@@
 	(wire
 		(pts
+			(xy 83.82 96.52) (xy 91.44 96.52)
+		)
+		(stroke
+			(width 0)
+			(type default)
+		)
+	)
+	(wire
+		(pts
 			(xy 234.95 165.1) (xy 236.22 165.1)
 		)
@@
 		)
 	)
+	(label "L_KEY22"
+		(at 106.68 96.52 180)
+		(effects
+			(font
+				(size 1.27 1.27)
+			)
+			(justify right bottom)
+		)
+	)
 	(label "L_KEY13"
 		(at 139.7 144.78 0)
@@
 		)
 	)
+	(label "KEY_18"
+		(at 83.82 96.52 0)
+		(effects
+			(font
+				(size 1.27 1.27)
+			)
+			(justify left bottom)
+		)
+	)
 	(label "L_KEY16"
 		(at 177.8 220.98 0)
@@
 		(unit 1)
 		(exclude_from_sim no)
-		(in_bom yes)
+		(in_bom no)
 		(on_board yes)
-		(dnp no)
+		(dnp yes)
 		(fields_autoplaced yes)
 		(property "Reference" "rU4"
@@
 	)
 	(symbol
+		(lib_id "Device:R")
+		(at 95.25 96.52 270)
+		(mirror x)
+		(unit 1)
+		(exclude_from_sim no)
+		(in_bom no)
+		(on_board yes)
+		(dnp yes)
+		(property "Reference" "rR19"
+			(at 95.25 93.98 90)
+			(effects
+				(font
+					(size 1.27 1.27)
+				)
+			)
+		)
+		(property "Value" "0R"
+			(at 95.25 99.06 90)
+			(effects
+				(font
+					(size 1.27 1.27)
+				)
+			)
+		)
+		(property "Footprint" "Resistor_SMD:R_0603_1608Metric"
+			(at 95.25 98.298 90)
+			(effects
+				(font
+					(size 1.27 1.27)
+				)
+				(hide yes)
+			)
+		)
+		(property "Datasheet" "~"
+			(at 95.25 96.52 0)
+			(effects
+				(font
+					(size 1.27 1.27)
+				)
+				(hide yes)
+			)
+		)
+		(property "Description" "Resistor"
+			(at 95.25 96.52 0)
+			(effects
+				(font
+					(size 1.27 1.27)
+				)
+				(hide yes)
+			)
+		)
+		(property "LCSC_Part" "C25804"
+			(at 95.25 96.52 90)
+			(effects
+				(font
+					(size 1.27 1.27)
+				)
+				(hide yes)
+			)
+		)
+		(property "Manufacturer_Name" "MULTICOMP PRO"
+			(at 95.25 96.52 90)
+			(effects
+				(font
+					(size 1.27 1.27)
+				)
+				(hide yes)
+			)
+		)
+		(property "Manufacturer_Name_1" ""
+			(at 95.25 96.52 90)
+			(effects
+				(font
+					(size 1.27 1.27)
+				)
+				(hide yes)
+			)
+		)
+		(property "Manufacturer_Name_2" "UNI-ROYAL(Uniroyal Elec)"
+			(at 95.25 96.52 90)
+			(effects
+				(font
+					(size 1.27 1.27)
+				)
+				(hide yes)
+			)
+		)
+		(property "Manufacturer_Part_Number" "MCWR06X1002FTL"
+			(at 95.25 96.52 90)
+			(effects
+				(font
+					(size 1.27 1.27)
+				)
+				(hide yes)
+			)
+		)
+		(property "Manufacturer_Part_Number_1" ""
+			(at 95.25 96.52 90)
+			(effects
+				(font
+					(size 1.27 1.27)
+				)
+				(hide yes)
+			)
+		)
+		(property "Manufacturer_Part_Number_2" "0603WAF1002T5E"
+			(at 95.25 96.52 90)
+			(effects
+				(font
+					(size 1.27 1.27)
+				)
+				(hide yes)
+			)
+		)
+		(pin "1"
+		)
+		(pin "2"
+		)
+		(instances
+			(project "corne-inidan-hotswap"
+				(path "/c90c0725-f1d3-4c5d-9757-c1f2f2a5449f/c662f5df-c1ad-47b5-b30e-5a138a045676"
+					(reference "rR19")
+					(unit 1)
+				)
+			)
+		)
+	)
+	(symbol
 		(lib_id "Device:C_Small")
 		(at 330.2 40.64 180)
@@
 		(unit 1)
 		(exclude_from_sim no)
-		(in_bom yes)
+		(in_bom no)
 		(on_board yes)
-		(dnp no)
+		(dnp yes)
 		(fields_autoplaced yes)
 		(property "Reference" "rJ1"
