File: pcbs/corne-indian/corne-inidan-hotswap/USB_HUB.kicad_sch (KiCad schematic)
At the start: 35 parts, among them J4 USB_A, J5 USB4105 - Type C USB 2.0 Conn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, J6 USB_A, J7 USB_A, J8 USB_A, Q1 SI2301, U5 CH334F, Y2 12Mhz

Commit message: USB Hub design updated
Parts:
- removed R12: 5K6, Resistor_SMD:R_0603_1608Metric, symbol Device:R
- added D10, D11, D7, D8, D9: LED, LED_SMD:LED_0603_1608Metric, symbol Device:LED
- added R16, R17: 5K1, Resistor_SMD:R_0603_1608Metric, symbol Device:R
- added R18: 0R/DNP, Resistor_SMD:R_0603_1608Metric, symbol Device:R_US
Connections:
- net GND: no longer R13.1
- net H+3.3V: now also D11.2 (A)
- net LED4: now reaches U5.21 (LED4/SDA)
- net LED4: now also R18.2
- net LED1: now reaches U5.22 (LED1)
- net LED1: now also R17.2
- net LED2: now reaches U5.23 (LED2)
- net LED2: now also R16.2
- net USB_VBUS_PIN: no longer names the net of R13.2
- net USB_VBUS_PIN: now also D10.2 (A), D7.1 (K), D8.2 (A), D9.1 (K), R18.1
- new net: D10.1 (K), D9.2 (A), R16.1
- new net: D7.2 (A), D8.1 (K), R17.1
- new net: D11.1 (K), R13.1
Other:
- moved on the sheet: R13
